Commit message: gazebo urdf colour added

File: fleet_interfaces/trolly/urdf/urdf.xacro (robot description, xacro)
@@ -15,5 +15,5 @@
         <box size="0.140 0.140 0.143"/>
       </geometry>
-      <material name="light_black"/>
+      <material name="orange"/>
     </visual>
     <collision>
@@ -31,4 +31,7 @@
     </inertial>
   </link>
+  <gazebo reference="base_link">
+    <material>Gazebo/Orange</material>
+  </gazebo>
   <joint name="wheel_left_joint" type="continuous">
     <parent link="base_link"/>
@@ -59,4 +62,7 @@
       </inertial>
   </link>
+  <gazebo reference="wheel_left_link">
+    <material>Gazebo/Red</material>
+  </gazebo>
   <joint name="wheel_right_joint" type="continuous">
     <parent link="base_link"/>
@@ -87,4 +93,7 @@
       </inertial>
   </link>
+  <gazebo reference="wheel_right_link">
+    <material>Gazebo/Red</material>
+  </gazebo>
   <joint name="caster_back_joint" type="fixed">
     <parent link="base_link"/>
@@ -107,4 +116,7 @@
     </inertial>
   </link>
+  <gazebo reference="caster_back_link">
+    <material>Gazebo/Red</material>
+  </gazebo>
   <joint name="imu_joint" type="fixed">
     <parent link="base_link"/>
@@ -113,4 +125,7 @@
   </joint>
   <link name="imu_link"/>
+  <gazebo reference="imu_link">
+    <material>Gazebo/Blue</material>
+  </gazebo>
   <joint name="scan_joint" type="fixed">
     <parent link="base_link"/>
@@ -140,3 +155,6 @@
     </inertial>
   </link>
+  <gazebo reference="base_scan">
+    <material>Gazebo/Blue</material>
+  </gazebo>
 </robot>
