Commit message: AMCL publishes map tf listening to /map

File: fleet_interfaces/trolly/urdf/urdf_double.xacro (robot description, xacro)
@@ -7,18 +7,18 @@
     <parent link="base_footprint"/>
     <child link="base_link"/>
-    <origin xyz="0.0 0.0 0.030" rpy="0 0 0"/>
+    <origin xyz="0.0 0.0 0.010" rpy="0 0 0"/>
   </joint>
   <link name="base_link">
     <visual>
-      <origin xyz="-0.096 0 0.210" rpy="0 0 0"/>
+      <origin xyz="-0.064 0 0.140" rpy="0 0 0"/>
       <geometry>
-        <box size="0.420 0.420 0.429"/>
+        <box size="0.280 0.280 0.286"/>
       </geometry>
       <material name="orange"/>
     </visual>
     <collision>
-      <origin xyz="-0.096 0 0.210" rpy="0 0 0"/>
+      <origin xyz="-0.064 0 0.140" rpy="0 0 0"/>
       <geometry>
-        <box size="0.420 0.420 0.429"/>
+        <box size="0.280 0.280 0.286"/>
       </geometry>
     </collision>
@@ -37,5 +37,5 @@
     <parent link="base_link"/>
     <child link="wheel_left_link"/>
-    <origin xyz="0.0 0.24 0.069" rpy="-1.57 0 0"/>
+    <origin xyz="0.0 0.16 0.046" rpy="-1.57 0 0"/>
     <axis xyz="0 0 1"/>
   </joint>
@@ -44,5 +44,5 @@
       <origin xyz="0 0 0" rpy="0 0 0"/>
       <geometry>
-        <cylinder length="0.054" radius="0.099"/>
+        <cylinder length="0.036" radius="0.066"/>
       </geometry>
       <material name="red"/>
@@ -51,5 +51,5 @@
       <origin xyz="0 0 0" rpy="0 0 0"/>
       <geometry>
-        <cylinder length="0.054" radius="0.099"/>
+        <cylinder length="0.036" radius="0.066"/>
       </geometry>
     </collision>
@@ -68,5 +68,5 @@
     <parent link="base_link"/>
     <child link="wheel_right_link"/>
-    <origin xyz="0.0 -0.240 0.069" rpy="-1.57 0 0"/>
+    <origin xyz="0.0 -0.160 0.046" rpy="-1.57 0 0"/>
     <axis xyz="0 0 1"/>
   </joint>
@@ -75,5 +75,5 @@
       <origin xyz="0 0 0" rpy="0 0 0"/>
       <geometry>
-        <cylinder length="0.054" radius="0.099"/>
+        <cylinder length="0.036" radius="0.066"/>
       </geometry>
       <material name="blue"/>
@@ -82,5 +82,5 @@
       <origin xyz="0 0 0" rpy="0 0 0"/>
       <geometry>
-        <cylinder length="0.054" radius="0.099"/>
+        <cylinder length="0.036" radius="0.066"/>
       </geometry>
     </collision>
@@ -99,11 +99,11 @@
     <parent link="base_link"/>
     <child link="caster_back_link"/>
-    <origin xyz="-0.243 0 -0.012" rpy="-1.57 0 0"/>
+    <origin xyz="-0.162 0 -0.008" rpy="-1.57 0 0"/>
   </joint>
   <link name="caster_back_link">
     <collision>
-      <origin xyz="0 0.003 0" rpy="0 0 0"/>
+      <origin xyz="0 0.002 0" rpy="0 0 0"/>
       <geometry>
-        <box size="0.090 0.027 0.060"/>
+        <box size="0.060 0.018 0.040"/>
       </geometry>
     </collision>
@@ -122,5 +122,5 @@
     <parent link="base_link"/>
     <child link="imu_link"/>
-    <origin xyz="-0.096 0 0.204" rpy="0 0 0"/>
+    <origin xyz="-0.064 0 0.136" rpy="0 0 0"/>
   </joint>
   <link name="imu_link"/>
@@ -131,17 +131,17 @@
     <parent link="base_link"/>
     <child link="base_scan"/>
-    <origin xyz="-0.096 0 0.516" rpy="0 0 0"/>
+    <origin xyz="-0.064 0 0.344" rpy="0 0 0"/>
   </joint>
   <link name="base_scan">
     <visual>
-      <origin xyz="0.045 0 -0.0195" rpy="0 0 0"/>
+      <origin xyz="0.030 0 -0.0130" rpy="0 0 0"/>
       <geometry>
-        <cylinder length="0.0945" radius="0.165"/>
+        <cylinder length="0.0630" radius="0.110"/>
       </geometry>
     </visual>
     <collision>
-      <origin xyz="0.045 0 -0.0195" rpy="0 0 0"/>
+      <origin xyz="0.030 0 -0.0130" rpy="0 0 0"/>
       <geometry>
-        <cylinder length="0.0945" radius="0.165"/>
+        <cylinder length="0.0630" radius="0.110"/>
       </geometry>
     </collision>

File: fleet_interfaces/trolly/urdf/urdf_single.xacro (robot description, xacro)
@@ -7,18 +7,18 @@
     <parent link="base_footprint"/>
     <child link="base_link"/>
-    <origin xyz="0.0 0.0 0.030" rpy="0 0 0"/>
+    <origin xyz="0.0 0.0 0.010" rpy="0 0 0"/>
   </joint>
   <link name="base_link">
     <visual>
-      <origin xyz="-0.096 0 0.210" rpy="0 0 0"/>
+      <origin xyz="-0.032 0 0.070" rpy="0 0 0"/>
       <geometry>
-        <box size="0.420 0.420 0.429"/>
+        <box size="0.140 0.140 0.143"/>
       </geometry>
       <material name="orange"/>
     </visual>
     <collision>
-      <origin xyz="-0.096 0 0.210" rpy="0 0 0"/>
+      <origin xyz="-0.032 0 0.070" rpy="0 0 0"/>
       <geometry>
-        <box size="0.420 0.420 0.429"/>
+        <box size="0.140 0.140 0.143"/>
       </geometry>
     </collision>
@@ -37,5 +37,5 @@
     <parent link="base_link"/>
     <child link="wheel_left_link"/>
-    <origin xyz="0.0 0.24 0.069" rpy="-1.57 0 0"/>
+    <origin xyz="0.0 0.08 0.023" rpy="-1.57 0 0"/>
     <axis xyz="0 0 1"/>
   </joint>
@@ -44,5 +44,5 @@
       <origin xyz="0 0 0" rpy="0 0 0"/>
       <geometry>
-        <cylinder length="0.054" radius="0.099"/>
+        <cylinder length="0.018" radius="0.033"/>
       </geometry>
       <material name="red"/>
@@ -51,5 +51,5 @@
       <origin xyz="0 0 0" rpy="0 0 0"/>
       <geometry>
-        <cylinder length="0.054" radius="0.099"/>
+        <cylinder length="0.018" radius="0.033"/>
       </geometry>
     </collision>
@@ -68,5 +68,5 @@
     <parent link="base_link"/>
     <child link="wheel_right_link"/>
-    <origin xyz="0.0 -0.240 0.069" rpy="-1.57 0 0"/>
+    <origin xyz="0.0 -0.080 0.023" rpy="-1.57 0 0"/>
     <axis xyz="0 0 1"/>
   </joint>
@@ -75,5 +75,5 @@
       <origin xyz="0 0 0" rpy="0 0 0"/>
       <geometry>
-        <cylinder length="0.054" radius="0.099"/>
+        <cylinder length="0.018" radius="0.033"/>
       </geometry>
       <material name="blue"/>
@@ -82,5 +82,5 @@
       <origin xyz="0 0 0" rpy="0 0 0"/>
       <geometry>
-        <cylinder length="0.054" radius="0.099"/>
+        <cylinder length="0.018" radius="0.033"/>
       </geometry>
     </collision>
@@ -99,11 +99,11 @@
     <parent link="base_link"/>
     <child link="caster_back_link"/>
-    <origin xyz="-0.243 0 -0.012" rpy="-1.57 0 0"/>
+    <origin xyz="-0.081 0 -0.004" rpy="-1.57 0 0"/>
   </joint>
   <link name="caster_back_link">
     <collision>
-      <origin xyz="0 0.003 0" rpy="0 0 0"/>
+      <origin xyz="0 0.001 0" rpy="0 0 0"/>
       <geometry>
-        <box size="0.090 0.027 0.060"/>
+        <box size="0.030 0.009 0.020"/>
       </geometry>
     </collision>
@@ -122,5 +122,5 @@
     <parent link="base_link"/>
     <child link="imu_link"/>
-    <origin xyz="-0.096 0 0.204" rpy="0 0 0"/>
+    <origin xyz="-0.032 0 0.068" rpy="0 0 0"/>
   </joint>
   <link name="imu_link"/>
@@ -131,17 +131,18 @@
     <parent link="base_link"/>
     <child link="base_scan"/>
-    <origin xyz="-0.096 0 0.516" rpy="0 0 0"/>
+    <origin xyz="-0.032 0 0.172" rpy="0 0 0"/>
   </joint>
   <link name="base_scan">
     <visual>
-      <origin xyz="0.045 0 -0.0195" rpy="0 0 0"/>
+      <origin xyz="0.015 0 -0.0065" rpy="0 0 0"/>
       <geometry>
-        <cylinder length="0.0945" radius="0.165"/>
+        <cylinder length="0.0315" radius="0.055"/>
       </geometry>
+      <material name="dark"/>
     </visual>
     <collision>
-      <origin xyz="0.045 0 -0.0195" rpy="0 0 0"/>
+      <origin xyz="0.015 0 -0.0065" rpy="0 0 0"/>
       <geometry>
-        <cylinder length="0.0945" radius="0.165"/>
+        <cylinder length="0.0315" radius="0.055"/>
       </geometry>
     </collision>
