Commit message: MoveBase prep

File: fleet_interfaces/trolly/urdf/urdf_triple.xacro (robot description, xacro)
@@ -137,11 +137,12 @@
       <origin xyz="0.045 0 -0.0195" rpy="0 0 0"/>
       <geometry>
-        <cylinder length="0.0945" radius="0.165"/>
+        <cylinder length="0.0315" radius="0.055"/>
       </geometry>
+      <material name="dark"/>
     </visual>
     <collision>
       <origin xyz="0.045 0 -0.0195" rpy="0 0 0"/>
       <geometry>
-        <cylinder length="0.0945" radius="0.165"/>
+        <cylinder length="0.0315" radius="0.055"/>
       </geometry>
     </collision>
