Commit message: Realignment of laserscan for triple trolly

File: fleet_interfaces/trolly/urdf/coloured_materials.xacro (robot description, xacro)
@@ -13,4 +13,7 @@
   <material name="blue">
     <color rgba="0.0 0.0 0.8 1.0"/>
+  </material>
+  <material name="yellow">
+    <color rgba="1.0 1.0 0.0 1.0"/>
   </material>
   <material name="green">

File: fleet_interfaces/trolly/urdf/urdf_single.xacro (robot description, xacro)
@@ -77,5 +77,5 @@
         <cylinder length="0.018" radius="0.033"/>
       </geometry>
-      <material name="blue"/>
+      <material name="red"/>
     </visual>
     <collision>
@@ -125,11 +125,8 @@
   </joint>
   <link name="imu_link"/>
-  <gazebo reference="imu_link">
-    <material>Gazebo/Blue</material>
-  </gazebo>
   <joint name="scan_joint" type="fixed">
     <parent link="base_link"/>
     <child link="base_scan"/>
-    <origin xyz="-0.032 0 0.172" rpy="0 0 0"/>
+    <origin xyz="-0.032 0 0.155" rpy="0 0 0"/>
   </joint>
   <link name="base_scan">
@@ -139,5 +136,5 @@
         <cylinder length="0.0315" radius="0.055"/>
       </geometry>
-      <material name="dark"/>
+      <material name="green"/>
     </visual>
     <collision>
@@ -156,5 +153,5 @@
   </link>
   <gazebo reference="base_scan">
-    <material>Gazebo/Blue</material>
+    <material>Gazebo/Green</material>
   </gazebo>
 </robot>

File: fleet_interfaces/trolly/urdf/urdf_triple.xacro (robot description, xacro)
@@ -11,14 +11,14 @@
   <link name="base_link">
     <visual>
-      <origin xyz="-0.096 0 0.210" rpy="0 0 0"/>
+      <origin xyz="-0.096 0 0.265" rpy="0 0 0"/>
       <geometry>
-        <box size="0.420 0.420 0.429"/>
+        <box size="0.420 0.420 0.530"/>
       </geometry>
       <material name="orange"/>
     </visual>
     <collision>
-      <origin xyz="-0.096 0 0.210" rpy="0 0 0"/>
+      <origin xyz="-0.096 0 0.265" rpy="0 0 0"/>
       <geometry>
-        <box size="0.420 0.420 0.429"/>
+        <box size="0.420 0.420 0.530"/>
       </geometry>
     </collision>
@@ -77,5 +77,5 @@
         <cylinder length="0.054" radius="0.099"/>
       </geometry>
-      <material name="blue"/>
+      <material name="red"/>
     </visual>
     <collision>
@@ -125,22 +125,19 @@
   </joint>
   <link name="imu_link"/>
-  <gazebo reference="imu_link">
-    <material>Gazebo/Blue</material>
-  </gazebo>
   <joint name="scan_joint" type="fixed">
     <parent link="base_link"/>
     <child link="base_scan"/>
-    <origin xyz="-0.096 0 0.516" rpy="0 0 0"/>
+    <origin xyz="-0.096 0 0.54575" rpy="0 0 0"/>
   </joint>
   <link name="base_scan">
     <visual>
-      <origin xyz="0.045 0 -0.0195" rpy="0 0 0"/>
+      <origin xyz="0.045 0 -0.01575" rpy="0 0 0"/>
       <geometry>
         <cylinder length="0.0315" radius="0.055"/>
       </geometry>
-      <material name="dark"/>
+      <material name="yellow"/>
     </visual>
     <collision>
-      <origin xyz="0.045 0 -0.0195" rpy="0 0 0"/>
+      <origin xyz="0.045 0 -0.01575" rpy="0 0 0"/>
       <geometry>
         <cylinder length="0.0315" radius="0.055"/>
@@ -156,5 +153,5 @@
   </link>
   <gazebo reference="base_scan">
-    <material>Gazebo/Blue</material>
+    <material>Gazebo/Yellow</material>
   </gazebo>
 </robot>
